File: 3D Printer Heated Bed/Heated Bed New.sch (EAGLE design)
At the start: 18 parts, among them IC1 7805T, IC2 ATMEGA168-20P, Q1 16Mhz, Q2 IRF530, X1 1751248, X2 1751248, X3 1751248

Commit message: Update
Parts:
- added J1: AVR_SPI_PRG_6PTH, SparkFun-Connectors:AVR_SPI_PRG_6PTH
- IC1: value 7805T -> 7805TV; device linear:7805T -> linear:7805TV
- LED1, LED2: value (none) -> 5
Connections:
- removed net GNDA: C1.1, C2.2, C3.-, C4.-, IC1.GND, OK2.EMIT, Q2.S, R2.2, R3.1, X1-1.K
- new net MISO: IC2.(PCI4/MISO)PB4, J1.1
- new net MOSI: IC2.(PCI3/MOSI/OC2A)PB3, J1.4
- new net RESET: IC2.PC6(/RESET/PCI14), J1.5
- new net SCK: IC2.(PCI5/SCK)PB5, J1.3
- net 5V: now also J1.2
- net ATMEGA_A0: now also IC2.(PCI8/ADC0)PC0
- net ATMEGA_D10: now also IC2.(PCI2/SS/OC1B)PB2
- net GND: now also C1.1, C2.2, C3.-, C4.-, IC1.GND, J1.6, OK2.EMIT, Q2.S, R2.2, R3.1, X1-1.K
