File: 3D Printer Heated Bed/Heated Bed.sch (EAGLE design)
At the start: 18 parts, among them IC1 7805T, IC2 ATMEGA168-20P, Q1 16Mhz, Q2 IRF530, X1 1751248, X2 1751248, X3 1751248

Commit message: Update
Connections:
- removed net GNDA: C1.1, C2.2, C3.-, C4.-, IC1.GND, OK2.EMIT, Q2.S, R2.2, R3.1, X1-1.K
- net GND: now also C1.1, C2.2, C3.-, C4.-, IC1.GND, OK2.EMIT, Q2.S, R2.2, R3.1, X1-1.K
